Commit message: Creat core URDF

File: description/robot.urdf.xacro (robot description, xacro)
@@ -2,3 +2,5 @@
 <robot xmlns:xacro="http://www.ros.org/wiki/xacro"  name="robot">
 <xacro:include filename="robot_core.xacro"/>
+<xacro:include filename="gazebo_control.xacro"/>
+<xacro:include filename="lidar.xacro" />
 </robot>

File: description/robot_core.xacro (robot description, xacro)
@@ -13,4 +13,7 @@
     <material name="black">
         <color rgba="0 0 0 1"/>
+    </material>
+    <material name="red">
+        <color rgba="1 0 0 1"/>
     </material>
     <!--BASE LINK-->
@@ -38,4 +41,7 @@
         </xacro:inertial_cylinder>
     </link>
+    <gazebo reference="chassis">
+        <material>Gazebo/White</material>
+    </gazebo>
     <!---->
     <joint name="chassis_joint" type="fixed">
@@ -48,5 +54,5 @@
     <parent link="base_link"/>
     <child link="left_wheel"/>
-    <origin xyz="0.15 0.15 0" rpy="-${pi/2} 0 0"/>
+    <origin xyz="0.11 0.11 0" rpy="-${pi/2} 0 0"/>ros2 run teleop_twist_keyboard teleop_twist_keyboard
     <axis xyz="0 0 1"/>
 </joint>
@@ -55,5 +61,5 @@
     <visual>
         <geometry>
-            <cylinder length="0.04" radius="0.05" />
+            <cylinder length="0.02" radius="0.05" />
         </geometry>
         <material name="blue"/>
@@ -62,17 +68,20 @@
     <collision>
         <geometry>
-            <cylinder length="0.04" radius="0.05" />
+            <cylinder length="0.02" radius="0.05" />
         </geometry>
     </collision>
     <!---->
-    <xacro:inertial_cylinder mass="0.05" length="0.04" radius="0.05">
+    <xacro:inertial_cylinder mass="0.05" length="0.02" radius="0.05">
         <origin xyz="0 0 0" rpy="0 0 0"/>
     </xacro:inertial_cylinder>
 </link>
+<gazebo reference="left_wheel">
+    <material>Gazebo/Blue</material>
+</gazebo>
      <!-- RIGHT WHEEL -->
 <joint name="right_wheel_joint" type="continuous">
     <parent link="base_link"/>
     <child link="right_wheel"/>
-    <origin xyz="0.15 -0.15 0" rpy="${pi/2} 0 0"/>
+    <origin xyz="0.11 -0.11 0" rpy="${pi/2} 0 0"/>
     <axis xyz="0 0 -1"/>
 </joint>
@@ -81,5 +90,5 @@
     <visual>
         <geometry>
-            <cylinder length="0.04" radius="0.05" />
+            <cylinder length="0.02" radius="0.05" />
         </geometry>
         <material name="blue"/>
@@ -88,12 +97,15 @@
     <collision>
         <geometry>
-            <cylinder length="0.04" radius="0.05" />
+            <cylinder length="0.02" radius="0.05" />
         </geometry>
     </collision>
      <!---->
-     <xacro:inertial_cylinder mass="0.05" length="0.04" radius="0.05">
+     <xacro:inertial_cylinder mass="0.05" length="0.02" radius="0.05">
         <origin xyz="0 0 0" rpy="0 0 0"/>
     </xacro:inertial_cylinder>
 </link>
+<gazebo reference="right_wheel">
+    <material>Gazebo/Blue</material>
+</gazebo>
    <!-- CASTER WHEEL -->
 <joint name="caster_wheel_joint" type="fixed">
@@ -120,3 +132,8 @@
     </xacro:inertial_sphere>
 </link>
+<gazebo reference="caster_wheel">
+    <material>Gazebo/Black</material>
+    <mu1 value="0.001"/>
+    <mu2 value="0.001"/>
+</gazebo>
 </robot>
